File: baseboard/baseboard.kicad_sch (KiCad schematic)
At the start: 1 part, among them U1 PY32E407V1xT_START

Commit message: add pmod
Parts:
- added J1: ~, kicad8-2:Pmod_socket, symbol kicad8-2:Pmod_Socket
Changed lines of the file:
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@@
 	(paper "A4")
+	(symbol
+		(lib_id "kicad8-2:Pmod_Socket")
+		(at 222.885 58.42 0)
+		(unit 1)
+		(exclude_from_sim no)
+		(in_bom yes)
+		(on_board yes)
+		(dnp no)
+		(fields_autoplaced yes)
+		(property "Reference" "J1"
+			(at 224.155 48.26 0)
+			(effects
+				(font
+					(size 1.27 1.27)
+				)
+			)
+		)
+		(property "Value" "~"
+			(at 224.155 50.8 0)
+			(effects
+				(font
+					(size 1.27 1.27)
+				)
+			)
+		)
+		(property "Footprint" "kicad8-2:Pmod_socket"
+			(at 222.885 58.42 0)
+			(effects
+				(font
+					(size 1.27 1.27)
+				)
+				(hide yes)
+			)
+		)
+		(property "Datasheet" "~"
+			(at 222.885 58.42 0)
+			(effects
+				(font
+					(size 1.27 1.27)
+				)
+				(hide yes)
+			)
+		)
+		(property "Description" ""
+			(at 222.885 58.42 0)
+			(effects
+				(font
+					(size 1.27 1.27)
+				)
+				(hide yes)
+			)
+		)
+		(pin "4"
+		)
+		(pin "1"
+		)
+		(pin "2"
+		)
+		(pin "3"
+		)
+		(pin "6"
+		)
+		(pin "5"
+		)
+		(pin "7"
+		)
+		(pin "8"
+		)
+		(pin "10"
+		)
+		(pin "11"
+		)
+		(pin "12"
+		)
+		(pin "9"
+		)
+		(instances
+			(project ""
+				(path "/63f1276c-2bcd-40b4-a634-5a67cabeeda8"
+					(reference "J1")
+					(unit 1)
+				)
+			)
+		)
+	)
 	(symbol
 		(lib_id "New_Library:PY32E407V1xT_START")

Commit message: schematics
Parts:
- added D1, D2, D3, D4: LED, LED_SMD:LED_0603_1608Metric_Pad1.05x0.95mm_HandSolder, symbol Device:LED

Commit message: schematics
Parts:
- added C1: 0.33u, Capacitor_SMD:C_0603_1608Metric_Pad1.08x0.95mm_HandSolder, symbol Device:C
- added C2: 2.2u, Capacitor_SMD:C_0603_1608Metric_Pad1.08x0.95mm_HandSolder, symbol Device:C
- added IC1: ATA6561-GAQW-N, SOIC127P600X175-8N, symbol kicad9_samacsys:ATA6561-GAQW-N
- added IC2: NJM2845DL1-33-TE1, TO-252-3-L1, symbol samacsys:NJM2845DL1-33-TE1
- added J10: Conn_01x01_Pin, Connector_PinHeader_2.54mm:PinHeader_1x01_P2.54mm_Vertical, symbol Connector:Conn_01x01_Pin
- added J2, J3: ~, kicad8-2:Pmod_socket, symbol kicad8-2:Pmod_Socket
- added J9: A295-CTRPB-1, A295CTRPB1, symbol samacsys:A295-CTRPB-1
- added S1, S2, S3, S4: TVBP06-B043CW-B, TVBP06B043CWB, symbol kicad8:TVBP06-B043CW-B
Connections:
- net Pmod1_1: now reaches J1.1 (Pin_1)
- net Pmod1_8: now reaches J1.10 (Pin_10)
- net GND: now reaches J1.11 (Pin_11)
- net GND: now also J1.5 (Pin_5), U1.103 (GND), U1.23 (GND), U1.48 (GND), U1.63 (GND), U1.74 (GND), U1.99 (GND), C1.2, C2.2, IC1.2 (GND), IC2.3 (GND), J2.11 (Pin_11), J2.5 (Pin_5), J3.11 (Pin_11), J3.5 (Pin_5), J9.2, J9.MH1, J9.MH2
- net +3V3: now reaches J1.12 (Pin_12)
- net +3V3: now also J1.6 (Pin_6), U1.100 (VDD), U1.105 (VDD), U1.24 (VDD), U1.49 (VDD), U1.64 (VDD), U1.75 (VDD), C2.1, IC1.5 (VIO), IC2.2 (VOUT), J2.12 (Pin_12), J2.6 (Pin_6), J3.12 (Pin_12), J3.6 (Pin_6)
- net Pmod1_2: now reaches J1.2 (Pin_2)
- net Pmod1_3: now reaches J1.3 (Pin_3)
- net Pmod1_4: now reaches J1.4 (Pin_4)
- net Pmod1_5: now reaches J1.7 (Pin_7)
- net Pmod1_6: now reaches J1.8 (Pin_8)
- net Pmod1_7: now reaches J1.9 (Pin_9)
- net at U1.60 (D13): now also IC1.8 (STBY)
- net at U1.82 (D0): now also IC1.4 (RXD)
- net at U1.83 (D1): now also IC1.1 (TXD)
- new net: C1.1, IC2.1 (VIN), J10.1 (Pin_1), J9.1
- new net +5V: IC1.3 (VCC)
- new net CANH: IC1.7 (CANH)
- new net CANL: IC1.6 (CANL)
- new net Pmod2_1: J2.1 (Pin_1)
- new net Pmod2_2: J2.2 (Pin_2)
- new net Pmod2_3: J2.3 (Pin_3)
- new net Pmod2_4: J2.4 (Pin_4)
- new net Pmod2_5: J2.7 (Pin_7)
- new net Pmod2_6: J2.8 (Pin_8)
- new net Pmod2_7: J2.9 (Pin_9)
- new net Pmod2_8: J2.10 (Pin_10)
- new net Pmod3_1: J3.1 (Pin_1)
- new net Pmod3_2: J3.2 (Pin_2)
- new net Pmod3_3: J3.3 (Pin_3)
- new net Pmod3_4: J3.4 (Pin_4)
- new net Pmod3_5: J3.7 (Pin_7)
- new net Pmod3_6: J3.8 (Pin_8)
- new net Pmod3_7: J3.9 (Pin_9)
- new net Pmod3_8: J3.10 (Pin_10)
Other:
- moved on the sheet: J1

Commit message: schematics
Parts:
- added VR1: RK09D117000B, RK09D117000B, symbol kicad9_samacsys:RK09D117000B
Changed lines of the file:
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@@
+	)
+	(symbol
+		(lib_id "kicad9_samacsys:RK09D117000B")
+		(at 234.315 65.405 0)
+		(unit 1)
+		(exclude_from_sim no)
+		(in_bom yes)
+		(on_board yes)
+		(dnp no)
+		(fields_autoplaced yes)
+		(property "Reference" "VR1"
+			(at 248.285 58.42 0)
+			(effects
+				(font
+					(size 1.27 1.27)
+				)
+			)
+		)
+		(property "Value" "RK09D117000B"
+			(at 248.285 60.96 0)
+			(effects
+				(font
+					(size 1.27 1.27)
+				)
+			)
+		)
+		(property "Footprint" "RK09D117000B"
+			(at 258.445 160.325 0)
+			(effects
+				(font
+					(size 1.27 1.27)
+				)
+				(justify left top)
+				(hide yes)
+			)
+		)
+		(property "Datasheet" "https://tech.alpsalpine.com/prod/j/html/potentiometer/rotarypotentiometers/rk09k/rk09d117000b.html"
+			(at 258.445 260.325 0)
+			(effects
+				(font
+					(size 1.27 1.27)
+				)
+				(justify left top)
+				(hide yes)
+			)
+		)
+		(property "Description" "9-inch insulated shaft snap-in type RK09K/RK09D series"
+			(at 234.315 65.405 0)
+			(effects
+				(font
+					(size 1.27 1.27)
+				)
+				(hide yes)
+			)
+		)
+		(property "Height" "30"
+			(at 258.445 460.325 0)
+			(effects
+				(font
+					(size 1.27 1.27)
+				)
+				(justify left top)
+				(hide yes)
+			)
+		)
+		(property "RS Part Number" ""
+			(at 258.445 560.325 0)
+			(effects
+				(font
+					(size 1.27 1.27)
+				)
+				(justify left top)
+				(hide yes)
+			)
+		)
+		(property "RS Price/Stock" ""
+			(at 258.445 660.325 0)
+			(effects
+				(font
+					(size 1.27 1.27)
+				)
+				(justify left top)
+				(hide yes)
+			)
+		)
+		(property "Manufacturer_Name" "ALPS Electric"
+			(at 258.445 760.325 0)
+			(effects
+				(font
+					(size 1.27 1.27)
+				)
+				(justify left top)
+				(hide yes)
+			)
+		)
+		(property "Manufacturer_Part_Number" "RK09D117000B"
+			(at 258.445 860.325 0)
+			(effects
+				(font
+					(size 1.27 1.27)
+				)
+				(justify left top)
+				(hide yes)
+			)
+		)
+		(pin "MH1"
+		)
+		(pin "MH2"
+		)
+		(pin "3"
+		)
+		(pin "1"
+		)
+		(pin "2"
+		)
+		(instances
+			(project ""
+				(path "/63f1276c-2bcd-40b4-a634-5a67cabeeda8"
+					(reference "VR1")
+					(unit 1)
+				)
+			)
+		)
 	)
 	(symbol
