File: baseboard/baseboard.kicad_sch (KiCad schematic)
At the start: 41 parts, among them IC1 ATA6561-GAQW-N, IC2 NJM2845DL1-33-TE1, J10 Conn_01x01_Pin, J11 Conn_01x02_Pin, J13 Conn_02x05_Odd_Even, J14 Conn_02x25_Odd_Even, J6 Screw_Terminal_01x02, J7 Conn_02x25_Odd_Even, J8 Conn_01x02_Pin, J9 A295-CTRPB-1, U1 PY32E407V1xT_START

Commit message: artwork done
Parts:
- removed C1: 0.33u, Capacitor_SMD:C_0603_1608Metric_Pad1.08x0.95mm_HandSolder, symbol Device:C
- removed C2: 2.2u, Capacitor_SMD:C_0603_1608Metric_Pad1.08x0.95mm_HandSolder, symbol Device:C
- removed IC2: NJM2845DL1-33-TE1, TO-252-3-L1, symbol samacsys:NJM2845DL1-33-TE1
- removed J10: Conn_01x01_Pin, Connector_PinHeader_2.54mm:PinHeader_1x01_P2.54mm_Vertical, symbol Connector:Conn_01x01_Pin
- removed J9: A295-CTRPB-1, A295CTRPB1, symbol samacsys:A295-CTRPB-1
- removed VR1: RK09D117000B, RK09D117000B, symbol kicad9_samacsys:RK09D117000B
- added S5: DTS-63N-V, DTS63NV, symbol kicad9_samacsys:DTS-63N-V
- D5: footprint samacsys:SM24CANB02HTG -> kicad9_samacsys:SM24CANB02HTG
- IC1: footprint SOIC127P600X175-8N -> kicad9_samacsys:SOIC127P600X175-8N
- L1: footprint samacsys:SDCW32162222TF -> kicad9_samacsys:SDCW32162222TF
- S1, S2, S3, S4: footprint TVBP06B043CWB -> kicad8:TVBP06B043CWB
Connections:
- net +3V3: now also J4.12 (Pin_12), J4.6 (Pin_6), J5.12 (Pin_12), J5.6 (Pin_6)
- net +5V: now also U1.106 (5V)
- net A11: now also J2.2 (Pin_2)
- net B15: now also IC1.8 (STBY)
- net C6: now also R10.2, S4.1 (COM); no longer R7.2, S1.1 (COM)
- net C7: now also R9.2, S3.1 (COM); no longer R8.2, S2.1 (COM)
- net C8: now also J3.3 (Pin_3); no longer R9.2, S3.1 (COM)
- net C9: now also J3.4 (Pin_4); no longer R10.2, S4.1 (COM)
- net D13: now also R7.2, S1.1 (COM); no longer IC1.8 (STBY)
- net D14: now also R8.2, S2.1 (COM)
- net ETH_MDC: now also J5.1 (Pin_1); no longer J5.2 (Pin_2)
- net ETH_MDIO: now also J14.22 (Pin_22), J5.2 (Pin_2); no longer J14.21 (Pin_21), J5.1 (Pin_1)
- net ETH_RMII_REF_CLK: now also J14.21 (Pin_21); no longer J14.22 (Pin_22)
- net GND: now also J4.11 (Pin_11), J4.5 (Pin_5), J5.11 (Pin_11), J5.5 (Pin_5), U1.110 (GND), S5.1 (COM_1)
- net Pmod1_1: now also J14.1 (Pin_1), U1.1 (E2); no longer J7.47 (Pin_47), U1.97 (E0)
- net Pmod1_2: now also J7.47 (Pin_47), U1.97 (E0); no longer J7.48 (Pin_48), U1.98 (E1)
- net Pmod1_3: now also J7.48 (Pin_48), U1.98 (E1); no longer J14.1 (Pin_1), U1.1 (E2)
- net Pmod2_1: now also J7.12 (Pin_12), U1.62 (D15); no longer J14.11 (Pin_11), U1.11 (F4)
- net Pmod2_3: now also J7.21 (Pin_21), U1.71 (A10); no longer J14.46 (Pin_46), U1.46 (E15)
- net Pmod2_4: now also J14.11 (Pin_11), U1.11 (F4); no longer J7.12 (Pin_12), U1.62 (D15)
- net Pmod2_5: now also J14.46 (Pin_46), U1.46 (E15); no longer J7.21 (Pin_21), U1.71 (A10)
- net Pmod3_1: now also J7.39 (Pin_39), U1.89 (D7); no longer J7.35 (Pin_35), U1.85 (D3)
- net Pmod3_2: now also J7.43 (Pin_43), U1.93 (B6); no longer J7.36 (Pin_36), U1.86 (D4)
- net Pmod3_5: now also J7.35 (Pin_35), U1.85 (D3); no longer J7.39 (Pin_39), U1.89 (D7)
- net Pmod3_6: now also J7.37 (Pin_37), U1.87 (D5); no longer J7.41 (Pin_41), U1.91 (B4)
- net Pmod3_7: now also J7.38 (Pin_38), U1.88 (D6); no longer J7.42 (Pin_42), U1.92 (B5)
- net Pmod3_8: now also J7.36 (Pin_36), U1.86 (D4); no longer J7.43 (Pin_43), U1.93 (B6)
- removed net Pmod2_2: J14.19 (Pin_19), J2.2 (Pin_2), U1.19 (F2)
- removed net Pmod3_3: J3.3 (Pin_3), J7.37 (Pin_37), U1.87 (D5)
- removed net Pmod3_4: J3.4 (Pin_4), J7.38 (Pin_38), U1.88 (D6)
- new net: S5.3 (NO_1), U1.111 (NRST)
- new net B4: J7.41 (Pin_41), U1.91 (B4)
- new net B5: J7.42 (Pin_42), U1.92 (B5)
- new net F2: U1.19 (F2)
- new net WIPER: J14.19 (Pin_19)
- no-connect marks 3 -> 6

Commit message: artwork confirm
Connections:
- net WIPER is gone; now on net F2: J14.19 (Pin_19)
Changed lines of the file:
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@@
-		)
-	)
-	(label "WIPER"
-		(at 230.505 60.325 0)
-		(effects
-			(font
-				(size 1.27 1.27)
-			)
-			(justify left bottom)
 		)
 	)
@@
 		(effects
 			(font
+				(size 1.27 1.27)
+			)
+			(justify left bottom)
+		)
+	)
+	(label "F2"
+		(at 230.505 60.325 0)
+		(effects
+			(font

Commit message: plot
Connections:
- net at D5.2, J11.2 (Pin_2), L1.3: now also J6.2 (Pin_2); no longer J6.1 (Pin_1)
- net at D5.1, J8.1 (Pin_1), L1.2: now also J6.1 (Pin_1); no longer J6.2 (Pin_2)
Other:
- moved on the sheet: J6
Changed lines of the file:
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@@
 	(wire
 		(pts
+			(xy 29.21 215.265) (xy 29.21 211.455)
+		)
+		(stroke
+			(width 0)
+			(type default)
+		)
+	)
+	(wire
+		(pts
 			(xy 146.05 205.105) (xy 150.495 205.105)
 		)
@@
 	(wire
 		(pts
+			(xy 29.21 205.105) (xy 29.21 208.915)
+		)
+		(stroke
+			(width 0)
+			(type default)
+		)
+	)
+	(wire
+		(pts
 			(xy 228.6 32.385) (xy 230.505 32.385)
 		)
@@
 	(wire
 		(pts
+			(xy 20.32 215.265) (xy 29.21 215.265)
+		)
+		(stroke
+			(width 0)
+			(type default)
+		)
+	)
+	(wire
+		(pts
 			(xy 137.16 64.77) (xy 139.7 64.77)
 		)
@@
 	(wire
 		(pts
+			(xy 20.32 208.915) (xy 20.32 205.105)
+		)
+		(stroke
+			(width 0)
+			(type default)
+		)
+	)
+	(wire
+		(pts
 			(xy 180.975 164.465) (xy 184.785 164.465)
 		)
@@
 	(wire
 		(pts
+			(xy 20.32 211.455) (xy 20.32 215.265)
+		)
+		(stroke
+			(width 0)
+			(type default)
+		)
+	)
+	(wire
+		(pts
 			(xy 139.7 85.09) (xy 137.16 85.09)
 		)
@@
 	(wire
 		(pts
+			(xy 20.32 205.105) (xy 29.21 205.105)
+		)
+		(stroke
+			(width 0)
+			(type default)
+		)
+	)
+	(wire
+		(pts
 			(xy 257.175 127.635) (xy 258.445 127.635)
 		)
@@
 	(symbol
 		(lib_id "Connector:Screw_Terminal_01x02")
-		(at 24.13 211.455 180)
+		(at 25.4 208.915 0)
 		(unit 1)
 		(exclude_from_sim no)
@@
 		(on_board yes)
 		(dnp no)
-		(fields_autoplaced yes)
 		(property "Reference" "J6"
-			(at 24.13 203.2 0)
+			(at 22.86 216.535 0)
 			(effects
 				(font
 					(size 1.27 1.27)
 				)
+				(justify left)
 			)
 		)
 		(property "Value" "Screw_Terminal_01x02"
-			(at 24.13 205.74 0)
+			(at 18.415 217.805 0)
 			(effects
 				(font
 					(size 1.27 1.27)
 				)
+				(justify left)
 			)
 		)
 		(property "Footprint" "TerminalBlock_Phoenix:TerminalBlock_Phoenix_MKDS-1,5-2-5.08_1x02_P5.08mm_Horizontal"
-			(at 24.13 211.455 0)
+			(at 25.4 208.915 0)
 			(effects
 				(font
@@
 		)
 		(property "Datasheet" "~"
-			(at 24.13 211.455 0)
+			(at 25.4 208.915 0)
 			(effects
 				(font
@@
 		)
 		(property "Description" "Generic screw terminal, single row, 01x02, script generated (kicad-library-utils/schlib/autogen/connector/)"
-			(at 24.13 211.455 0)
+			(at 25.4 208.915 0)
 			(effects
 				(font

Commit message: add t1s on baseboard
Parts:
- removed J4, J5: ~, kicad8-2:Pmod_socket, symbol kicad8-2:Pmod_Socket
- added C10, C13, C16, C4, C5, C7: 0.1u, Capacitor_SMD:C_0603_1608Metric_Pad1.08x0.95mm_HandSolder, symbol Device:C
- added C11, C14, C9: 10u, Capacitor_SMD:C_0805_2012Metric_Pad1.18x1.45mm_HandSolder, symbol Device:C
- added C12, C15, C6, C8: 10000p, Capacitor_SMD:C_0603_1608Metric_Pad1.08x0.95mm_HandSolder, symbol Device:C
- added C2, C3: 0.22u, Capacitor_SMD:C_0603_1608Metric_Pad1.08x0.95mm_HandSolder, symbol Device:C
- added FL1: ACT1210E-131-2P-TL00, ACT1210E1312PTL00, symbol samacsys:ACT1210E-131-2P-TL00
- added IC2: LAN8670C2-E_LMX, QFN50P500X500X100-33N-D, symbol samacsys:LAN8670C2-E_LMX
- added J7: Screw_Terminal_01x02, TerminalBlock_MetzConnect:TerminalBlock_MetzConnect_Type055_RT01502HDWU_1x02_P5.00mm_Horizontal, symbol Connector:Screw_Terminal_01x02
- added J8, J9: Conn_01x02_Pin, Connector_PinHeader_2.54mm:PinHeader_1x02_P2.54mm_Vertical, symbol Connector:Conn_01x02_Pin
- added L2, L3: 300R, symbol Device:L
- added R10, R11, R12, R17, R18, R19, R30, R31, R33, R34, R35, R36, R37, R5, R6, R7, R8, R9: 10k, Resistor_SMD:R_0603_1608Metric_Pad0.98x0.95mm_HandSolder, symbol Device:R
- added R24, R25, R32: 4.7k, Resistor_SMD:R_0603_1608Metric_Pad0.98x0.95mm_HandSolder, symbol Device:R
- added R26, R28, R29: 22, Resistor_SMD:R_0603_1608Metric_Pad0.98x0.95mm_HandSolder, symbol Device:R
- added R27: 12.4k, Resistor_SMD:R_0603_1608Metric_Pad0.98x0.95mm_HandSolder, symbol Device:R
- added R3, R4: 49.9, Resistor_SMD:R_0603_1608Metric_Pad0.98x0.95mm_HandSolder, symbol Device:R
- added RV1, RV2: AVRH10C221KT1R5YA8, RESC1005X55N, symbol samacsys:AVRH10C221KT1R5YA8
- added Y1: CB3LV-3C-50M0000, CB3LV3C50M0000, symbol samacsys:CB3LV-3C-50M0000
- renumbered C3 to C1, D5 to D1, D1 to D2, D2 to D3, D3 to D4, D4 to D5, J6 to J1, J1 to J10, J12 to J11, J2 to J12, J3 to J13, J8 to J2, J11 to J3, J13 to J4, J7 to J5, J14 to J6, R3 to R13, R4 to R14, R5 to R15, R6 to R16, R7 to R20, R8 to R21, R9 to R22, R10 to R23, S5 to S1, S1 to S2, S2 to S3, S3 to S4, S4 to S5
Connections:
- net ETH_RMII_REF_CLK is gone; now on net ETH_MDIO: J6.21 (Pin_22), U1.21 (A2)
- net +3V3: now also J6.23 (Pin_24), J6.50 (Pin_49), U1.23 (VDD), U1.50 (VDD), C12.1, C13.1, C14.1, C15.2, C16.2, IC2.18 (VDDP_2), IC2.8 (VDDP_1), L3.2, R18.2, R24.2, R25.2, R30.2, R32.2, R37.2, Y1.4 (VCC); no longer J6.24 (Pin_24), J6.49 (Pin_49), U1.24 (VDD), U1.49 (VDD)
- net A0: now also J6.19 (Pin_20), U1.19 (A0); no longer J6.20 (Pin_20), U1.20 (A0)
- net A3: now also J6.26 (Pin_25), U1.26 (A3); no longer J6.25 (Pin_25), U1.25 (A3)
- net A4: now also J6.25 (Pin_26), U1.25 (A4); no longer J6.26 (Pin_26), U1.26 (A4)
- net A5: now also J6.28 (Pin_27), U1.28 (A5); no longer J6.27 (Pin_27), U1.27 (A5)
- net A6: now also J6.27 (Pin_28), U1.27 (A6); no longer J6.28 (Pin_28), U1.28 (A6)
- net A7: now also J6.30 (Pin_29), U1.30 (A7); no longer J6.29 (Pin_29), U1.29 (A7)
- net B0: now also J6.31 (Pin_32), U1.31 (B0); no longer J6.32 (Pin_32), U1.32 (B0)
- net B1: now also J6.34 (Pin_33), U1.34 (B1); no longer J6.33 (Pin_33), U1.33 (B1)
- net B10: now also J6.48 (Pin_47), U1.48 (B10); no longer J6.47 (Pin_47), U1.47 (B10)
- net C0: now also J6.16 (Pin_15), U1.16 (C0); no longer J6.15 (Pin_15), U1.15 (C0)
- net C13: now also J6.8 (Pin_7), U1.8 (C13); no longer J6.7 (Pin_7), U1.7 (C13)
- net C14: now also J6.7 (Pin_8), U1.7 (C14); no longer J6.8 (Pin_8), U1.8 (C14)
- net C15: now also J6.10 (Pin_9), U1.10 (C15); no longer J6.9 (Pin_9), U1.9 (C15)
- net C2: now also J6.18 (Pin_17), U1.18 (C2); no longer J6.17 (Pin_17), U1.17 (C2)
- net C3: now also J6.17 (Pin_18), U1.17 (C3); no longer J6.18 (Pin_18), U1.18 (C3)
- net C4: now also J6.29 (Pin_30), U1.29 (C4); no longer J6.30 (Pin_30), U1.30 (C4)
- net C5: now also J6.32 (Pin_31), U1.32 (C5); no longer J6.31 (Pin_31), U1.31 (C5)
- net ETH_MDC: now also J6.15 (Pin_16), U1.15 (C1), IC2.13 (MDC), R24.1; no longer J6.16 (Pin_16), U1.16 (C1)
- net ETH_MDIO: now also IC2.14 (MDIO), R25.1; no longer J6.22 (Pin_22), U1.22 (A2)
- net ETH_RMII_CRS_DV: now also IC2.20 (RXDV_/_CRSDV_/_PHYAD1), R34.1
- net ETH_RMII_RXD0: now also R26.1, R9.2
- net ETH_RMII_RXD1: now also R29.2, R35.1
- net ETH_RMII_TXD0: now also IC2.6 (TXD0)
- net ETH_RMII_TXD1: now also IC2.5 (TXD1)
- net ETH_RMII_TX_EN: now also J6.49 (Pin_50), U1.49 (B11), IC2.7 (TXEN), R6.1; no longer J6.50 (Pin_50), U1.50 (B11)
- net F0: now also J6.11 (Pin_12), U1.11 (F0); no longer J6.12 (Pin_12), U1.12 (F0)
- net F1: now also J6.14 (Pin_13), U1.14 (F1); no longer J6.13 (Pin_13), U1.13 (F1)
- net F2: now also J6.20 (Pin_19), U1.20 (F2); no longer J6.19 (Pin_19), U1.19 (F2)
- net F3: now also J6.9 (Pin_10), U1.9 (F3); no longer J6.10 (Pin_10), U1.10 (F3)
- net F5: now also J6.13 (Pin_14), U1.13 (F5); no longer J6.14 (Pin_14), U1.14 (F5)
- net GND: now also J6.24 (Pin_23), J6.47 (Pin_48), U1.24 (GND), U1.47 (GND), C10.1, C11.1, C12.2, C13.2, C14.2, C15.1, C16.1, C6.1, C7.1, C8.1, C9.1, IC2.3 (TXD3), IC2.33 (VSS), IC2.4 (TXD2), J8.2 (Pin_2), J9.1 (Pin_1), R10.1, R11.1, R12.2, R17.1, R27.2, R31.2, R33.2, R34.2, R35.2, R36.2, R5.2, R6.2, R7.2, R8.1, R9.1, RV1.2, RV2.2, Y1.2 (GND); no longer J6.23 (Pin_23), J6.48 (Pin_48), U1.23 (GND), U1.48 (GND)
- net Pmod1_1: now also J6.2 (Pin_1), U1.2 (E2); no longer J6.1 (Pin_1), U1.1 (E2)
- net Pmod1_4: now also J6.1 (Pin_2), U1.1 (E3); no longer J6.2 (Pin_2), U1.2 (E3)
- net Pmod1_5: now also J6.4 (Pin_3), U1.4 (E4); no longer J6.3 (Pin_3), U1.3 (E4)
- net Pmod1_6: now also J6.3 (Pin_4), U1.3 (E5); no longer J6.4 (Pin_4), U1.4 (E5)
- net Pmod1_7: now also J6.6 (Pin_5), U1.6 (E6); no longer J6.5 (Pin_5), U1.5 (E6)
- net Pmod1_8: now also J6.46 (Pin_45), U1.46 (E14); no longer J6.45 (Pin_45), U1.45 (E14)
- net Pmod2_4: now also J6.12 (Pin_11), U1.12 (F4); no longer J6.11 (Pin_11), U1.11 (F4)
- net Pmod2_5: now also J6.45 (Pin_46), U1.45 (E15); no longer J6.46 (Pin_46), U1.46 (E15)
- net Pmod4_1: now also J6.33 (Pin_34), U1.33 (B2); no longer J6.34 (Pin_34), U1.34 (B2)
- net Pmod4_2: now also J6.37 (Pin_38), U1.37 (E7); no longer J6.38 (Pin_38), U1.38 (E7)
- net Pmod4_3: now also J6.40 (Pin_39), U1.40 (E8); no longer J6.39 (Pin_39), U1.39 (E8)
- net Pmod4_4: now also J6.39 (Pin_40), U1.39 (E9); no longer J6.40 (Pin_40), U1.40 (E9)
- net Pmod4_5: now also J6.42 (Pin_41), U1.42 (E10); no longer J6.41 (Pin_41), U1.41 (E10)
- net Pmod4_6: now also J6.41 (Pin_42), U1.41 (E11); no longer J6.42 (Pin_42), U1.42 (E11)
- net Pmod4_7: now also J6.44 (Pin_43), U1.44 (E12); no longer J6.43 (Pin_43), U1.43 (E12)
- net Pmod4_8: now also J6.43 (Pin_44), U1.43 (E13); no longer J6.44 (Pin_44), U1.44 (E13)
- net VBAT: now also J6.5 (Pin_6), U1.5 (VBAT), L2.2; no longer J6.6 (Pin_6), U1.6 (VBAT)
- net VCCA: now also J6.38 (Pin_37), U1.38 (VCCA); no longer J6.37 (Pin_37), U1.37 (VCCA)
- net VREF+: now also J6.35 (Pin_36), U1.35 (VREF+); no longer J6.36 (Pin_36), U1.36 (VREF+)
- net VSSA: now also J6.36 (Pin_35), U1.36 (VSSA); no longer J6.35 (Pin_35), U1.35 (VSSA)
- new net: C5.1, J7.2 (Pin_2), R4.1, R7.1, RV2.1
- new net: C3.2, R4.2
- new net: C4.1, J7.1 (Pin_1), R3.1, R5.1, RV1.1
- new net: C4.2, FL1.3
- new net: IC2.16 (RXD0_/_PHYAD2), R26.2
- new net: IC2.19 (RXD1_/_PHYAD3), R29.1
- new net: IC2.2 (COL), R17.2
- new net: IC2.21 (RXER_/_PHYAD0), R28.1
- new net: C5.2, FL1.4
- new net: R37.1, Y1.1 (EOH)
- new net: C3.1, J9.2 (Pin_2)
- new net: C2.1, J8.1 (Pin_1)
- new net: C2.2, R3.2
- new net ACMA: IC2.11 (TXER_/_ACMA), R11.2
- new net CLK50M: IC2.27 (XTI_/_REFCLKIN), J6.22 (Pin_21), U1.22 (A1), Y1.3 (OUTPUT)
- new net GPIO0: IC2.9 (GPIO0), R8.2
- new net INH: IC2.1 (INH), R12.1
- new net Mode0: IC2.23 (RXD2_/_MODE0), R31.1
- new net Mode1: IC2.24 (RXD3_/_MODE1), R30.1
- new net PHYAD4: IC2.15 (CRS_/_PHYAD4), R10.2
- new net RBIAS: IC2.26 (RBIAS), R27.1
- new net RXER: R28.2, R33.1
- new net RXPI: IC2.12 (TXCLK_/_RXPI)
- new net TRX_N: FL1.1, IC2.31 (TRXN)
- new net TRX_P: FL1.2, IC2.30 (TRXP)
- new net VDDA: C6.2, C7.2, C9.2, IC2.29 (VDDA), L3.1
- new net VDDAU: C10.2, C11.2, C8.2, IC2.25 (VDDAU), L2.1, R19.2
- new net WAKE_IN: IC2.32 (WAKE_IN), R19.1
- new net WAKE_OUT: IC2.17 (RXCLK_/_SMCLK_/_WAKE_OUT), R36.1
- new net nINT: IC2.22 (IRQ_N), R32.1
- new net nRST: IC2.10 (RESET_N), R18.1
- no-connect marks 6 -> 7

Commit message: schematics
Parts:
- added R38, R39: 22, Resistor_SMD:R_0603_1608Metric_Pad0.98x0.95mm_HandSolder, symbol Device:R
Connections:
- net B7: now also R22.2, S4.1 (COM)
- net B9: now also R23.2, S5.1 (COM)
- net C13: now also R21.2, S3.1 (COM)
- net C14: no longer J6.7 (Pin_8)
- net C15: no longer J6.10 (Pin_9)
- net C6: no longer R23.2, S5.1 (COM)
- net C7: no longer R22.2, S4.1 (COM)
- net CLK50M: now also R39.2; no longer J6.22 (Pin_21), U1.22 (A1), Y1.3 (OUTPUT)
- net D13: no longer R20.2, S2.1 (COM)
- net D14: no longer R21.2, S3.1 (COM)
- net F3: now also R20.2, S2.1 (COM)
- new net: R38.2, R39.1, Y1.3 (OUTPUT)
- new net ETH_RMII_REF_CLK: J6.22 (Pin_21), R38.1, U1.22 (A1)
Changed lines of the file:
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@@
 	)
 	(junction
+		(at 462.28 -48.26)
+		(diameter 0)
+		(color 0 0 0 0)
+	)
+	(junction
 		(at 338.455 -21.59)
 		(diameter 0)
@@
 	)
 	(junction
-		(at 447.04 -48.26)
-		(diameter 0)
-		(color 0 0 0 0)
-	)
-	(junction
 		(at 319.405 120.015)
 		(diameter 0)
@@
 	(wire
 		(pts
-			(xy 257.175 249.555) (xy 259.08 249.555)
+			(xy 462.28 -38.735) (xy 462.28 -36.83)
 		)
 		(stroke
@@
 	(wire
 		(pts
-			(xy 412.75 2.54) (xy 415.925 2.54)
+			(xy 257.175 249.555) (xy 259.08 249.555)
 		)
 		(stroke
@@
 	(wire
 		(pts
-			(xy 212.725 83.185) (xy 215.9 83.185)
+			(xy 412.75 2.54) (xy 415.925 2.54)
 		)
 		(stroke
@@
 	(wire
 		(pts
-			(xy 184.785 250.825) (xy 172.72 250.825)
+			(xy 212.725 83.185) (xy 215.9 83.185)
 		)
 		(stroke
@@
 	(wire
 		(pts
-			(xy 208.28 24.765) (xy 208.28 86.995)
+			(xy 184.785 250.825) (xy 172.72 250.825)
 		)
 		(stroke
@@
 	(wire
 		(pts
-			(xy 257.175 193.675) (xy 280.67 193.675)
+			(xy 208.28 24.765) (xy 208.28 86.995)
 		)
 		(stroke
@@
 	(wire
 		(pts
-			(xy 212.725 75.565) (xy 215.9 75.565)
+			(xy 257.175 193.675) (xy 280.67 193.675)
 		)
 		(stroke
@@
 	(wire
 		(pts
+			(xy 447.04 -48.26) (xy 462.28 -48.26)
+		)
+		(stroke
+			(width 0)
+			(type default)
+		)
+	)
+	(wire
+		(pts
 			(xy 332.74 210.185) (xy 332.74 199.39)
 		)
@@
 	(wire
 		(pts
-			(xy 446.405 -48.26) (xy 447.04 -48.26)
-		)
-		(stroke
-			(width 0)
-			(type default)
-		)
-	)
-	(wire
-		(pts
 			(xy 137.16 82.55) (xy 139.7 82.55)
 		)
@@
 	(wire
 		(pts
-			(xy 228.6 73.025) (xy 230.505 73.025)
-		)
-		(stroke
-			(width 0)
-			(type default)
-		)
-	)
-	(wire
-		(pts
 			(xy 373.38 -53.34) (xy 386.08 -53.34)
 		)
@@
 	(wire
 		(pts
+			(xy 462.28 -48.26) (xy 464.82 -48.26)
+		)
+		(stroke
+			(width 0)
+			(type default)
+		)
+	)
+	(wire
+		(pts
 			(xy 309.245 -43.18) (xy 313.055 -43.18)
 		)
@@
 	(wire
 		(pts
-			(xy 454.025 -36.83) (xy 351.155 -36.83)
+			(xy 462.28 -36.83) (xy 351.155 -36.83)
 		)
 		(stroke
@@
 	(wire
 		(pts
-			(xy 454.025 -48.26) (xy 454.025 -36.83)
+			(xy 462.28 -48.26) (xy 462.28 -46.355)
 		)
 		(stroke
@@
 	(wire
 		(pts
+			(xy 472.44 -48.26) (xy 474.98 -48.26)
+		)
+		(stroke
+			(width 0)
+			(type default)
+		)
+	)
+	(wire
+		(pts
 			(xy 287.02 64.77) (xy 287.02 67.945)
 		)
@@
 	(wire
 		(pts
-			(xy 447.04 -48.26) (xy 454.025 -48.26)
-		)
-		(stroke
-			(width 0)
-			(type default)
-		)
-	)
-	(wire
-		(pts
 			(xy 415.29 -54.61) (xy 415.29 -45.72)
 		)
@@
 		)
 	)
-	(label "C6"
-		(at 349.885 220.98 180)
-		(effects
-			(font
-				(size 1.27 1.27)
-			)
-			(justify right bottom)
-		)
-	)
 	(label "Pmod3_5"
 		(at 137.16 67.31 180)
@@
 		)
 	)
+	(label "ETH_RMII_REF_CLK"
+		(at 474.98 -48.26 0)
+		(effects
+			(font
+				(size 1.27 1.27)
+			)
+			(justify left bottom)
+		)
+	)
 	(label "VBAT"
 		(at 212.725 78.105 180)
@@
 		)
 	)
+	(label "B7"
+		(at 347.98 210.185 0)
+		(effects
+			(font
+				(size 1.27 1.27)
+			)
+			(justify left bottom)
+		)
+	)
 	(label "JTCK"
 		(at 137.16 57.15 180)
@@
 		)
 	)
-	(label "C7"
-		(at 349.885 210.185 180)
-		(effects
-			(font
-				(size 1.27 1.27)
-			)
-			(justify right bottom)
-		)
-	)
 	(label "B15"
 		(at 106.68 210.185 180)
@@
 		)
 	)
+	(label "F3"
+		(at 346.71 188.595 0)
+		(effects
+			(font
+				(size 1.27 1.27)
+			)
+			(justify left bottom)
+		)
+	)
+	(label "C13"
+		(at 347.345 199.39 0)
+		(effects
+			(font
+				(size 1.27 1.27)
+			)
+			(justify left bottom)
+		)
+	)
 	(label "Pmod4_7"
 		(at 230.505 29.845 0)
@@
 		)
 	)
-	(label "D14"
-		(at 347.345 199.39 0)
-		(effects
-			(font
-				(size 1.27 1.27)
-			)
-			(justify left bottom)
-		)
-	)
 	(label "CANL"
 		(at 112.395 205.105 180)
@@
 		)
 	)
-	(label "ETH_RMII_REF_CLK"
-		(at 454.025 -48.26 0)
-		(effects
-			(font
-				(size 1.27 1.27)
-			)
-			(justify left bottom)
-		)
-	)
 	(label "Pmod2_1"
 		(at 154.94 36.83 0)
@@
 		)
 	)
-	(label "D13"
-		(at 347.345 188.595 0)
-		(effects
-			(font
-				(size 1.27 1.27)
-			)
-			(justify left bottom)
-		)
-	)
 	(label "Pmod4_1"
 		(at 259.715 168.275 0)
@@
 		)
 	)
+	(label "B9"
+		(at 347.98 220.98 0)
+		(effects
+			(font
+				(size 1.27 1.27)
+			)
+			(justify left bottom)
+		)
+	)
 	(label "CAN_TXD"
 		(at 137.16 64.77 180)
@@
 	)
 	(symbol
+		(lib_id "Device:R")
+		(at 468.63 -48.26 270)
+		(unit 1)
+		(exclude_from_sim no)
+		(in_bom yes)
+		(on_board yes)
+		(dnp no)
+		(property "Reference" "R38"
+			(at 468.63 -45.72 90)
+			(effects
+				(font
+					(size 1.27 1.27)
+				)
+			)
+		)
+		(property "Value" "22"
+			(at 468.63 -48.26 90)
+			(effects
+				(font
+					(size 1.27 1.27)
+				)
+			)
+		)
+		(property "Footprint" "Resistor_SMD:R_0603_1608Metric_Pad0.98x0.95mm_HandSolder"
+			(at 468.63 -50.038 90)
+			(effects
+				(font
+					(size 1.27 1.27)
+				)
+				(hide yes)
+			)
+		)
+		(property "Datasheet" "~"
+			(at 468.63 -48.26 0)
+			(effects
+				(font
+					(size 1.27 1.27)
+				)
+				(hide yes)
+			)
+		)
+		(property "Description" "Resistor"
+			(at 468.63 -48.26 0)
+			(effects
+				(font
+					(size 1.27 1.27)
+				)
+				(hide yes)
+			)
+		)
+		(pin "1"
+		)
+		(pin "2"
+		)
+		(instances
+			(project "baseboard"
+				(path "/63f1276c-2bcd-40b4-a634-5a67cabeeda8"
+					(reference "R38")
+					(unit 1)
+				)
+			)
+		)
+	)
+	(symbol
 		(lib_id "power:GND")
 		(at 150.495 215.9 0)
@@
 					(unit 1)
 				)
+			)
+		)
+	)
+	(symbol
+		(lib_id "Device:R")
+		(at 462.28 -42.545 0)
+		(unit 1)
+		(exclude_from_sim no)
+		(in_bom yes)
+		(on_board yes)
+		(dnp no)
+		(property "Reference" "R39"
+			(at 464.82 -42.545 90)
+			(effects
+				(font
+					(size 1.27 1.27)
+				)
+			)
+		)
+		(property "Value" "22"
+			(at 462.28 -42.545 90)
+			(effects
+				(font
+					(size 1.27 1.27)
+				)
+			)
+		)
+		(property "Footprint" "Resistor_SMD:R_0603_1608Metric_Pad0.98x0.95mm_HandSolder"
+			(at 460.502 -42.545 90)
+			(effects
+				(font
+					(size 1.27 1.27)
+				)
+				(hide yes)
+			)
+		)
+		(property "Datasheet" "~"
+			(at 462.28 -42.545 0)
+			(effects
+				(font
+					(size 1.27 1.27)
+				)
+				(hide yes)
+			)
+		)
+		(property "Description" "Resistor"
+			(at 462.28 -42.545 0)
+			(effects
+				(font
+					(size 1.27 1.27)
+				)
+				(hide yes)
+			)
+		)
+		(pin "1"
+		)
+		(pin "2"
+		)
+		(instances
+			(project "baseboard"
+				(path "/63f1276c-2bcd-40b4-a634-5a67cabeeda8"
+					(reference "R39")
+					(unit 1)
+				)

Commit message: base baord schematics
Parts:
- FL1: footprint ACT1210E1312PTL00 -> kicad9_samacsys:ACT1210E1312PTL00
- IC2: footprint QFN50P500X500X100-33N-D -> kicad9_samacsys:QFN50P500X500X100-33N-D
- RV1, RV2: footprint RESC1005X55N -> kicad9_samacsys:RESC1005X55N
- S1: footprint DTS63NV -> kicad9_samacsys:DTS63NV
Changed lines of the file:
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@@
 			)
 		)
-		(property "Footprint" "QFN50P500X500X100-33N-D"
+		(property "Footprint" "kicad9_samacsys:QFN50P500X500X100-33N-D"
 			(at 370.205 80.95 0)
 			(effects
@@
 			)
 		)
-		(property "Footprint" "RESC1005X55N"
+		(property "Footprint" "kicad9_samacsys:RESC1005X55N"
 			(at 148.92 -27.305 0)
 			(effects
@@
 			)
 		)
-		(property "Footprint" "ACT1210E1312PTL00"
+		(property "Footprint" "kicad9_samacsys:ACT1210E1312PTL00"
 			(at 316.865 -140.005 0)
 			(effects
@@
 			)
 		)
-		(property "Footprint" "DTS63NV"
+		(property "Footprint" "kicad9_samacsys:DTS63NV"
 			(at 274.955 195.885 0)
 			(effects
@@
 			)
 		)
-		(property "Footprint" "RESC1005X55N"
+		(property "Footprint" "kicad9_samacsys:RESC1005X55N"
 			(at 157.81 -26.67 0)
 			(effects

Commit message: base board schematics
Connections:
- net Pmod1_5: now also J6.46 (Pin_45), U1.46 (E14); no longer J6.4 (Pin_3), U1.4 (E4)
- net Pmod1_8: now also J6.4 (Pin_3), U1.4 (E4); no longer J6.46 (Pin_45), U1.46 (E14)
- net Pmod4_1: now also J6.44 (Pin_43), U1.44 (E12); no longer J6.33 (Pin_34), U1.33 (B2)
- net Pmod4_2: now also J6.42 (Pin_41), U1.42 (E10); no longer J6.37 (Pin_38), U1.37 (E7)
- net Pmod4_5: now also J11.7 (Pin_7), J6.43 (Pin_44), U1.43 (E13); no longer J11.10 (Pin_10), J6.42 (Pin_41), U1.42 (E10)
- net Pmod4_6: now also J11.8 (Pin_8); no longer J11.9 (Pin_9)
- net Pmod4_7: now also J11.9 (Pin_9), J6.33 (Pin_34), U1.33 (B2); no longer J11.8 (Pin_8), J6.44 (Pin_43), U1.44 (E12)
- net Pmod4_8: now also J11.10 (Pin_10), J6.37 (Pin_38), U1.37 (E7); no longer J11.7 (Pin_7), J6.43 (Pin_44), U1.43 (E13)
