File: baseboard/baseboard.kicad_sch (KiCad schematic)
At the start: 88 parts, among them IC1 ATA6561-GAQW-N, IC2 LAN8670C2-E_LMX, J1 Screw_Terminal_01x02, J2 Conn_01x02_Pin, J3 Conn_01x02_Pin, J4 Conn_02x05_Odd_Even, J5 Conn_02x25_Odd_Even, J6 Conn_02x25_Odd_Even, J7 Screw_Terminal_01x02, J8 Conn_01x02_Pin, J9 Conn_01x02_Pin, U1 PY32E407V1xT_START, Y1 CB3LV-3C-50M0000

Commit message: base board schematics
Connections:
- net B4 is gone; now on net Pmod2_5: J5.41 (Pin_41), U1.91 (B4)
- net Pmod2_5: no longer J6.45 (Pin_46), U1.45 (E15)
- net Pmod3_6: now also J5.36 (Pin_36), U1.86 (D4); no longer J5.37 (Pin_37), U1.87 (D5)
- net Pmod3_7: now also J5.37 (Pin_37), U1.87 (D5); no longer J5.38 (Pin_38), U1.88 (D6)
- net Pmod3_8: now also J5.38 (Pin_38), U1.88 (D6); no longer J5.36 (Pin_36), U1.86 (D4)
- new net E15: J6.45 (Pin_46), U1.45 (E15)
Changed lines of the file:
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@@
 	(wire
 		(pts
+			(xy 182.88 222.885) (xy 184.785 222.885)
+		)
+		(stroke
+			(width 0)
+			(type default)
+		)
+	)
+	(wire
+		(pts
 			(xy 212.725 78.105) (xy 215.9 78.105)
 		)
@@
 	(wire
 		(pts
+			(xy 182.88 220.345) (xy 184.785 220.345)
+		)
+		(stroke
+			(width 0)
+			(type default)
+		)
+	)
+	(wire
+		(pts
 			(xy 241.935 -43.18) (xy 254 -43.18)
 		)
@@
 	(wire
 		(pts
+			(xy 257.175 137.795) (xy 259.715 137.795)
+		)
+		(stroke
+			(width 0)
+			(type default)
+		)
+	)
+	(wire
+		(pts
 			(xy 257.175 239.395) (xy 259.715 239.395)
 		)
@@
 	(wire
 		(pts
-			(xy 137.16 74.93) (xy 139.7 74.93)
-		)
-		(stroke
-			(width 0)
-			(type default)
-		)
-	)
-	(wire
-		(pts
 			(xy 449.58 -45.72) (xy 449.58 -1.27)
 		)
@@
 	(wire
 		(pts
+			(xy 212.725 27.305) (xy 215.9 27.305)
+		)
+		(stroke
+			(width 0)
+			(type default)
+		)
+	)
+	(wire
+		(pts
 			(xy 184.785 187.325) (xy 168.91 187.325)
 		)
@@
 	(wire
 		(pts
-			(xy 257.175 137.795) (xy 259.715 137.795)
-		)
-		(stroke
-			(width 0)
-			(type default)
-		)
-	)
-	(wire
-		(pts
 			(xy 212.725 57.785) (xy 215.9 57.785)
 		)
@@
 	(wire
 		(pts
-			(xy 182.88 220.345) (xy 184.785 220.345)
-		)
-		(stroke
-			(width 0)
-			(type default)
-		)
-	)
-	(wire
-		(pts
 			(xy 158.75 202.565) (xy 158.75 207.645)
 		)
@@
 	(wire
 		(pts
-			(xy 257.175 175.895) (xy 259.715 175.895)
+			(xy 137.16 74.93) (xy 139.7 74.93)
 		)
 		(stroke
@@
 	(wire
 		(pts
-			(xy 309.245 122.555) (xy 319.405 122.555)
+			(xy 257.175 175.895) (xy 259.715 175.895)
 		)
 		(stroke
@@
 	(wire
 		(pts
-			(xy 212.725 27.305) (xy 215.9 27.305)
+			(xy 309.245 122.555) (xy 319.405 122.555)
 		)
 		(stroke
@@
 	(wire
 		(pts
+			(xy 182.88 230.505) (xy 184.785 230.505)
+		)
+		(stroke
+			(width 0)
+			(type default)
+		)
+	)
+	(wire
+		(pts
 			(xy 299.72 146.05) (xy 301.625 146.05)
 		)
@@
 	(wire
 		(pts
-			(xy 182.88 217.805) (xy 184.785 217.805)
+			(xy 405.13 2.54) (xy 405.13 6.35)
 		)
 		(stroke
@@
 	(wire
 		(pts
-			(xy 405.13 2.54) (xy 405.13 6.35)
+			(xy 342.265 220.98) (xy 354.965 220.98)
 		)
 		(stroke
@@
 	(wire
 		(pts
-			(xy 342.265 220.98) (xy 354.965 220.98)
+			(xy 318.135 32.385) (xy 310.515 32.385)
 		)
 		(stroke
@@
 	(wire
 		(pts
-			(xy 318.135 32.385) (xy 310.515 32.385)
+			(xy 20.32 215.265) (xy 29.21 215.265)
 		)
 		(stroke
@@
 	(wire
 		(pts
-			(xy 20.32 215.265) (xy 29.21 215.265)
+			(xy 152.4 67.31) (xy 154.94 67.31)
 		)
 		(stroke
@@
 	(wire
 		(pts
+			(xy 137.16 69.85) (xy 139.7 69.85)
+		)
+		(stroke
+			(width 0)
+			(type default)
+		)
+	)
+	(wire
+		(pts
 			(xy 374.015 13.97) (xy 381 13.97)
 		)
@@
 	(wire
 		(pts
-			(xy 271.78 -17.78) (xy 271.78 -15.875)
+			(xy 152.4 69.85) (xy 154.94 69.85)
 		)
 		(stroke
@@
 	(wire
 		(pts
-			(xy 152.4 77.47) (xy 154.94 77.47)
+			(xy 271.78 -17.78) (xy 271.78 -15.875)
 		)
 		(stroke
@@
 	(wire
 		(pts
-			(xy 180.34 128.905) (xy 184.785 128.905)
+			(xy 152.4 77.47) (xy 154.94 77.47)
 		)
 		(stroke
@@
 	(wire
 		(pts
-			(xy 257.175 221.615) (xy 259.715 221.615)
+			(xy 180.34 128.905) (xy 184.785 128.905)
 		)
 		(stroke
@@
 	(wire
 		(pts
-			(xy 340.995 67.945) (xy 303.53 67.945)
+			(xy 257.175 221.615) (xy 259.715 221.615)
 		)
 		(stroke
@@
 	(wire
 		(pts
-			(xy 152.4 67.31) (xy 154.94 67.31)
+			(xy 340.995 67.945) (xy 303.53 67.945)
 		)
 		(stroke
@@
 	(wire
 		(pts
-			(xy 137.16 69.85) (xy 139.7 69.85)
-		)
-		(stroke
-			(width 0)
-			(type default)
-		)
-	)
-	(wire
-		(pts
 			(xy 180.34 133.985) (xy 184.785 133.985)
 		)
@@
 	(wire
 		(pts
-			(xy 152.4 69.85) (xy 154.94 69.85)
-		)
-		(stroke
-			(width 0)
-			(type default)
-		)
-	)
-	(wire
-		(pts
 			(xy 127.635 39.37) (xy 127.635 88.265)
 		)
@@
 	(wire
 		(pts
-			(xy 137.16 72.39) (xy 139.7 72.39)
+			(xy 182.88 217.805) (xy 184.785 217.805)
 		)
 		(stroke
@@
 	(wire
 		(pts
-			(xy 405.13 -14.605) (xy 405.13 -21.59)
+			(xy 137.16 72.39) (xy 139.7 72.39)
 		)
 		(stroke
@@
 	(wire
 		(pts
-			(xy 310.515 32.385) (xy 310.515 29.21)
+			(xy 405.13 -14.605) (xy 405.13 -21.59)
 		)
 		(stroke
@@
 	(wire
 		(pts
-			(xy 272.415 130.175) (xy 272.415 129.54)
+			(xy 310.515 32.385) (xy 310.515 29.21)
 		)
 		(stroke
@@
 	(wire
 		(pts
-			(xy 412.75 -5.715) (xy 415.925 -5.715)
+			(xy 272.415 130.175) (xy 272.415 129.54)
 		)
 		(stroke
@@
 	(wire
 		(pts
-			(xy 146.05 202.565) (xy 158.75 202.565)
+			(xy 412.75 -5.715) (xy 415.925 -5.715)
 		)
 		(stroke
@@
 	(wire
 		(pts
-			(xy 182.88 230.505) (xy 184.785 230.505)
+			(xy 146.05 202.565) (xy 158.75 202.565)
 		)
 		(stroke
@@
 	(wire
 		(pts
-			(xy 182.88 222.885) (xy 184.785 222.885)
-		)
-		(stroke
-			(width 0)
-			(type default)
-		)
-	)
-	(wire
-		(pts
 			(xy 335.915 52.07) (xy 335.915 55.245)
 		)
@@
 		)
 	)
-	(label "B4"
-		(at 182.88 230.505 180)
-		(effects
-			(font
-				(size 1.27 1.27)
-			)
-			(justify right bottom)
-		)
-	)
 	(label "ETH_RMII_RXD0"
 		(at 180.34 141.605 180)
@@
 	)
 	(label "Pmod3_7"
-		(at 182.88 222.885 180)
+		(at 182.88 220.345 180)
 		(effects
 			(font
@@
 		)
 	)
+	(label "E15"
+		(at 212.725 27.305 180)
+		(effects
+			(font
+				(size 1.27 1.27)
+			)
+			(justify right bottom)
+		)
+	)
 	(label "F2"
 		(at 230.505 60.325 0)
@@
 		)
 	)
+	(label "E15"
+		(at 259.715 137.795 0)
+		(effects
+			(font
+				(size 1.27 1.27)
+			)
+			(justify left bottom)
+		)
+	)
 	(label "A0"
 		(at 212.725 60.325 180)
@@
 	)
 	(label "Pmod3_8"
-		(at 154.94 67.31 0)
+		(at 154.94 69.85 0)
 		(effects
 			(font
@@
 	)
 	(label "Pmod3_8"
-		(at 182.88 217.805 180)
+		(at 182.88 222.885 180)
 		(effects
 			(font
@@
 	)
 	(label "Pmod3_7"
-		(at 154.94 69.85 0)
+		(at 137.16 69.85 180)
 		(effects
 			(font
 				(size 1.27 1.27)
 			)
-			(justify left bottom)
+			(justify right bottom)
 		)
 	)
@@
 		)
 	)
+	(label "Pmod2_5"
+		(at 137.16 74.93 180)
+		(effects
+			(font
+				(size 1.27 1.27)
+			)
+			(justify right bottom)
+		)
+	)
 	(label "ETH_RMII_RXD0"
 		(at 154.94 29.21 0)
@@
 	)
 	(label "Pmod2_5"
-		(at 259.715 137.795 0)
+		(at 182.88 230.505 180)
 		(effects
 			(font
 				(size 1.27 1.27)
 			)
-			(justify left bottom)
+			(justify right bottom)
 		)
 	)
@@
 		)
 	)
-	(label "Pmod2_5"
-		(at 212.725 27.305 180)
-		(effects
-			(font
-				(size 1.27 1.27)
-			)
-			(justify right bottom)
-		)
-	)
 	(label "Pmod2_6"
 		(at 182.245 200.025 180)
@@
 	)
 	(label "Pmod3_6"
-		(at 182.88 220.345 180)
+		(at 182.88 217.805 180)
 		(effects
 			(font
@@
 		)
 	)
-	(label "B4"
-		(at 137.16 74.93 180)
-		(effects
-			(font
-				(size 1.27 1.27)
-			)
-			(justify right bottom)
-		)
-	)
 	(label "VSSA"
 		(at 259.715 165.735 0)
@@
 	)
 	(label "Pmod3_6"
-		(at 137.16 69.85 180)
+		(at 154.94 67.31 0)
 		(effects
 			(font
 				(size 1.27 1.27)
 			)
-			(justify right bottom)
+			(justify left bottom)
 		)
 	)
