File: baseboard/baseboard.kicad_pcb (KiCad board)
At the start: 2 copper layers, 99.8 x 102.1 mm, 88 parts, among them IC1 ATA6561-GAQW-N, IC2 LAN8670C2-E_LMX, J1 Screw_Terminal_01x02, J2 Conn_01x02_Pin, J3 Conn_01x02_Pin, J4 Conn_02x05_Odd_Even, J5 Conn_02x25_Odd_Even, J6 Conn_02x25_Odd_Even, J7 Screw_Terminal_01x02, J8 Conn_01x02_Pin, J9 Conn_01x02_Pin, U1 PY32E407V1xT_START, Y1 CB3LV-3C-50M0000

Commit message: base board shcematics
Parts:
- added L2: 300R, Inductor_SMD:L_0603_1608Metric_Pad1.05x0.95mm_HandSolder, B.Cu at (125.9, 95.2)
- added L3: 300R, Inductor_SMD:L_0603_1608Metric_Pad1.05x0.95mm_HandSolder, F.Cu at (133.6, 82.8)
- added R40: 0, Resistor_SMD:R_0603_1608Metric_Pad0.98x0.95mm_HandSolder, F.Cu at (129.2, 93.7)
- C1, C10, C11, C12, C13, C14, C15, C16, C2, C3, C8, R1, R18, R19, R2, R27, R29, R3, R34, R35, R4, R5, R7: moved to B.Cu
- R6: value 10k -> 0
- moved R34 105.7 mm to (93.9, 91.4), turned to -90 degrees
- moved R35 105.7 mm to (93.9, 95.4), turned to 90 degrees
- moved R29 103.6 mm to (96.8, 96.4), turned to 180 degrees
- moved R26 98.6 mm to (96.9, 91.9)
- moved C14 98.6 mm to (109.7, 78.0), turned to 90 degrees
- moved R9 97.7 mm to (93.9, 91.1), turned to -90 degrees
- moved R11 92.5 mm to (102.6, 82.7), turned to 45 degrees
- moved R8 86.8 mm to (106.7, 79.0), turned to -90 degrees
- moved R36 85.9 mm to (114.4, 88.6), turned to 180 degrees
- moved R18 85.0 mm to (110.6, 81.2), turned to 180 degrees
- moved R10 81.6 mm to (111.6, 85.5)
- moved C11 81.5 mm to (123.3, 92.2)
- moved R37 80.8 mm to (118.9, 109.1), turned to 180 degrees
- moved R33 79.7 mm to (119.9, 98.0), turned to -90 degrees
- moved C13 79.2 mm to (112.1, 78.1), turned to 90 degrees
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Connections:
- C4 pad 1: Net-(J7-Pin_1) -> Net-(J7-Pin_2)
- C5 pad 1: Net-(J7-Pin_2) -> Net-(J7-Pin_1)
- IC1 pad 8: /B15 -> /B14
- IC2 pad 12: /RXPI -> unconnected-(IC2-TXCLK_/_RXPI-Pad12)
- J5 pad 16: /C7 -> /RXER
- J5 pad 4: /B15 -> /GPIO0
- R3 pad 1: Net-(J7-Pin_1) -> Net-(J7-Pin_2)
- R38 pad 1: /ETH_RMII_REF_CLK -> Net-(R38-Pad1)
- R39 pad 2: /CLK50M -> Net-(R39-Pad2)
- R4 pad 1: Net-(J7-Pin_2) -> Net-(J7-Pin_1)
- R5 pad 1: Net-(J7-Pin_1) -> Net-(J7-Pin_2)
- R6 pad 1: /ETH_RMII_TX_EN -> /ETH_RMII_REF_CLK
- R6 pad 2: GND -> Net-(R38-Pad1)
- R7 pad 1: Net-(J7-Pin_2) -> Net-(J7-Pin_1)
- RV1 pad 1: Net-(J7-Pin_1) -> Net-(J7-Pin_2)
- RV2 pad 1: Net-(J7-Pin_2) -> Net-(J7-Pin_1)
- U1 pad 54: /B15 -> /GPIO0
- U1 pad 66: /C7 -> /RXER
Routing:
- net +3V3: track 292.1 -> 469.9 mm, vias 1 -> 6
- net /ETH_MDC: track 8.44 -> 93.1 mm
- net /ETH_MDIO: track 8.44 -> 85.4 mm
- net /VBAT: track 8.44 -> 78.1 mm, vias 0 -> 2
- net /A6: track 8.44 -> 69.9 mm, vias 0 -> 1
- net /B15: track 52.2 -> 0.00 mm, vias 1 -> 0
- net /A5: track 8.44 -> 57.7 mm, vias 0 -> 1
- net /GPIO0: track 0.00 -> 47.4 mm, vias 0 -> 1
- net /A4: track 8.44 -> 55.7 mm, vias 0 -> 1
- net /RXER: track 0.00 -> 44.8 mm, vias 0 -> 1
- net /B14: track 8.67 -> 50.4 mm, vias 0 -> 1
- net /ETH_RMII_CRS_DV: track 8.67 -> 49.5 mm, vias 0 -> 1
- net /ETH_RMII_TXD0: track 8.67 -> 48.4 mm
- net /ETH_RMII_TX_EN: track 0.00 -> 39.0 mm, vias 0 -> 1
- net /ETH_RMII_TXD1: track 10.5 -> 48.9 mm
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Other:
- board size 99.8 x 102.1 mm -> 99.8 x 99.9 mm
- board text added: "CAN"
- board text added: "D|F"
- board text added: "Pmod EXP v0.2 for PY32E407 -START-ETH V2.1"
- board text added: "T1S"
- board text added: "VSSA|VREF"
- board text removed: "D2|F4"
- board text removed: "Pmod EXP v0.1 for PY32E407-START-ETH V2.1"
- board text removed: "VREF|VSSA"

Commit message: base board v0.2 done
Routing:
- net /Pmod4_8: track 32.1 -> 23.7 mm
- net /B14: track 50.4 -> 48.7 mm
- net /Pmod4_7: track 38.3 -> 37.2 mm
- net +3V3: track 469.9 -> 471.0 mm
- net GND: vias 125 -> 126
Other:
- board text added: "B1|B2"
- board text added: "C0|C1"
- board text added: "C10|A10"
- board text added: "C13|C14"
- board text added: "C15|F3"
- board text added: "C2|C3"
- board text added: "C6|C7"
- board text added: "C8|C9"
- board text added: "D12|D13"
- board text added: "D14|D15"
- board text added: "D15|F4"
- board text added: "D2|A11"
- board text added: "D3|D7"
- board text added: "D4|B6"
- board text added: "D5|C8"
- board text added: "D6|C9"
- board text added: "E2|E14"
- board text added: "E2|E3"
- board text added: "E3|E4"
- board text added: "E4|E5"
- board text added: "E6|VBAT"
- board text added: "F1|F5"
- board text added: "F2|A0"
- board text added: "F4|F0"
- board text added: "VCCA|E7"
- board text removed: "C10|A11"
- board text removed: "C12|A10"
- board text removed: "D|B"
- board text removed: "D|C"
- board text removed: "D|D"
- board text removed: "D|F"
- board text removed: "E2|E4"
- board text removed: "E3|E14"
