File: ether_board/LAN8670/LAN8671.kicad_sch (KiCad schematic)
At the start: 50 parts, among them IC1 LAN8670C2-E_LMX, J1 Screw_Terminal_01x02, J2 Conn_01x02_Pin, J3 Conn_01x02_Pin

Commit message: schematics
Parts:
- added J4, J5: ~, kicad8-2:Pmod, symbol kicad8-2:Pmod_Pin
Changed lines of the file:
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@@
+	)
+	(symbol
+		(lib_id "kicad8-2:Pmod_Pin")
+		(at 254 90.17 0)
+		(unit 1)
+		(exclude_from_sim no)
+		(in_bom yes)
+		(on_board yes)
+		(dnp no)
+		(fields_autoplaced yes)
+		(property "Reference" "J5"
+			(at 255.27 80.01 0)
+			(effects
+				(font
+					(size 1.27 1.27)
+				)
+			)
+		)
+		(property "Value" "~"
+			(at 255.27 82.55 0)
+			(effects
+				(font
+					(size 1.27 1.27)
+				)
+			)
+		)
+		(property "Footprint" "kicad8-2:Pmod"
+			(at 254 90.17 0)
+			(effects
+				(font
+					(size 1.27 1.27)
+				)
+				(hide yes)
+			)
+		)
+		(property "Datasheet" "~"
+			(at 254 90.17 0)
+			(effects
+				(font
+					(size 1.27 1.27)
+				)
+				(hide yes)
+			)
+		)
+		(property "Description" ""
+			(at 254 90.17 0)
+			(effects
+				(font
+					(size 1.27 1.27)
+				)
+				(hide yes)
+			)
+		)
+		(pin "3"
+		)
+		(pin "7"
+		)
+		(pin "9"
+		)
+		(pin "6"
+		)
+		(pin "11"
+		)
+		(pin "5"
+		)
+		(pin "1"
+		)
+		(pin "10"
+		)
+		(pin "8"
+		)
+		(pin "2"
+		)
+		(pin "4"
+		)
+		(pin "12"
+		)
+		(instances
+			(project "LAN8671"
+				(path "/94f51103-8592-4d9a-89d2-39ddc6afe3a4"
+					(reference "J5")
+					(unit 1)
+				)
+			)
+		)
 	)
 	(symbol
@@
 					(unit 1)
 				)
+			)
+		)
+	)
+	(symbol
+		(lib_id "kicad8-2:Pmod_Pin")
+		(at 253.365 54.61 0)
+		(unit 1)
+		(exclude_from_sim no)
+		(in_bom yes)
+		(on_board yes)
+		(dnp no)
+		(fields_autoplaced yes)
+		(property "Reference" "J4"
+			(at 254.635 44.45 0)
+			(effects
+				(font
+					(size 1.27 1.27)
+				)
+			)
+		)
+		(property "Value" "~"
+			(at 254.635 46.99 0)
+			(effects
+				(font
+					(size 1.27 1.27)
+				)
+			)
+		)
+		(property "Footprint" "kicad8-2:Pmod"
+			(at 253.365 54.61 0)
+			(effects
+				(font
+					(size 1.27 1.27)
+				)
+				(hide yes)
+			)
+		)
+		(property "Datasheet" "~"
+			(at 253.365 54.61 0)
+			(effects
+				(font
+					(size 1.27 1.27)
+				)
+				(hide yes)
+			)
+		)
+		(property "Description" ""
+			(at 253.365 54.61 0)
+			(effects
+				(font
+					(size 1.27 1.27)
+				)
+				(hide yes)
+			)
+		)
+		(pin "3"
+		)
+		(pin "7"
+		)
+		(pin "9"
+		)
+		(pin "6"
+		)
+		(pin "11"
+		)
+		(pin "5"
+		)
+		(pin "1"
+		)
+		(pin "10"
+		)
+		(pin "8"
+		)
+		(pin "2"
+		)
+		(pin "4"
+		)
+		(pin "12"
+		)
+		(instances
+			(project ""
+				(path "/94f51103-8592-4d9a-89d2-39ddc6afe3a4"
+					(reference "J4")
+					(unit 1)
+				)

Commit message: ether board schematics
Parts:
- added Y1: CB3LV-3C-50M0000, CB3LV3C50M0000, symbol samacsys:CB3LV-3C-50M0000
Connections:
- net +3V3: now also J4.12 (Pin_12), J4.6 (Pin_6), J5.12 (Pin_12), J5.6 (Pin_6)
- net ACMA: now also J5.10 (Pin_10)
- net CLK50M: now also J4.1 (Pin_1)
- net CRSDV: now also J4.7 (Pin_7)
- net GND: now also J4.11 (Pin_11), J4.5 (Pin_5), J5.11 (Pin_11), J5.5 (Pin_5)
- net GPIO0: now also J5.7 (Pin_7)
- net INH: now also J5.4 (Pin_4)
- net MDC: now also J5.1 (Pin_1)
- net MDIO: now also J5.2 (Pin_2)
- net RXD0: now also J4.2 (Pin_2)
- net RXD1: now also J4.8 (Pin_8)
- net RXER: now also J4.10 (Pin_10)
- net RXPI: now also J5.9 (Pin_9)
- net TXD0: now also J4.9 (Pin_9)
- net TXD1: now also J4.4 (Pin_4)
- net nINT: now also J5.8 (Pin_8)
- net nRST: now also J5.3 (Pin_3)
- net TXEN: now reaches J4.3 (Pin_3)
- net TXEN: now also IC1.7 (TXEN), R4.1
